File: PCB/test_schem_swaw.kicad_pcb (KiCad board)
At the start: 2 copper layers, 73.7 x 77.5 mm, 8 parts, among them J1 Jack-DC, J2 Conn_02x19_Counter_Clockwise, J3 Conn_01x06, J4 Conn_01x05, J5 Conn_02x19_Counter_Clockwise, J6 Conn_01x04, U1 DHT11

Commit message: Modified scheme of PCB - final version, not developed anymore
Parts:
- removed J1: Jack-DC, Connector_BarrelJack:BarrelJack_Horizontal
- added C2: 100n, Capacitor_THT:C_Disc_D7.5mm_W4.4mm_P5.00mm, F.Cu at (60.5, 66.0)
- C1: value CP -> 100n; footprint Capacitor_THT:CP_Radial_D5.0mm_P2.00mm -> Capacitor_THT:C_Disc_D7.5mm_W4.4mm_P5.00mm
- moved C1 26.6 mm to (45.0, 66.0), turned to 270 degrees
Connections:
- net GND renamed Net-(C1-Pad2)
- J2 pad 18: Net-(J2-Pad18) -> Net-(C1-Pad1)
- J2 pad 6: Net-(C1-Pad1) -> Net-(J2-Pad6)
- U1 pad 1: Net-(J2-Pad18) -> Net-(C1-Pad1)
Routing:
- net Net-(C1-Pad2): track 155.5 -> 1.44 mm
- net Net-(J4-Pad4): track 26.4 -> 51.4 mm
- net Net-(J2-Pad18): track 22.5 -> 0.00 mm
- net Net-(C1-Pad1): track 37.0 -> 28.7 mm
- net Net-(C2-Pad1): track 90.8 -> 85.3 mm
- net Net-(J5-Pad12): track 78.7 -> 81.8 mm
- net Net-(J5-Pad14): track 72.3 -> 73.4 mm
- net Net-(J3-Pad4): track 21.8 -> 22.5 mm
- added copper zone on In2.Cu, net Net-(C1-Pad1)
- added copper zone on B.Cu, net Net-(C1-Pad2)
- added copper zone on F.Cu, net Net-(C1-Pad2)
Other:
- board size 73.7 x 77.5 mm -> 78.7 x 71.1 mm
- copper layers 2 -> 4
