File: PCB/test_schem_swaw.sch (KiCad schematic (older format))
At the start: 8 parts, among them J1 Jack-DC, J2 Conn_02x19_Counter_Clockwise, J3 Conn_01x06, J4 Conn_01x05, J5 Conn_02x19_Counter_Clockwise, J6 Conn_01x04, U1 DHT11

Commit message: Modified scheme of PCB - final version, not developed anymore
Parts:
- removed C1: CP, Capacitor_THT:CP_Radial_D5.0mm_P2.00mm, symbol Device:CP
- removed J1: Jack-DC, Connector_BarrelJack:BarrelJack_Horizontal, symbol Connector:Jack-DC
- added C1, C2: 100n, Capacitor_THT:C_Disc_D7.5mm_W4.4mm_P5.00mm, symbol Device:C
Connections:
- net GND: no longer J2.22 (Pin_22), J3.5 (Pin_5), J4.2 (Pin_2), J6.3 (Pin_3), U1.4 (GND)
- net at J2.18 (Pin_18), U1.1 (VCC): now also C1.1
- net at J2.16 (Pin_16), J3.6 (Pin_6), J4.1 (Pin_1)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: now also C2.1
- new net: C1.2, C2.2, J2.22 (Pin_22), J3.5 (Pin_5), J4.2 (Pin_2), J6.3 (Pin_3), U1.4 (GND)
Changed lines of the file:
@@
 $EndComp
-$Comp
-L power:GND #PWR01
-U 1 1 60906A04
-P 3950 900
-F 0 "#PWR01" H 3950 650 50  0001 C CNN
-F 1 "GND" H 3955 727 50  0000 C CNN
-F 2 "" H 3950 900 50  0001 C CNN
-F 3 "" H 3950 900 50  0001 C CNN
-	1    3950 900
-	0    -1   1    0
-$EndComp
-Wire Wire Line
-	2800 1150 3200 1150
 $Comp
 L Connector_Generic:Conn_02x19_Odd_Even J2
@@
 $EndComp
 $Comp
-L Connector:Jack-DC J1
-U 1 1 609034C2
-P 2700 850
-F 0 "J1" H 2757 1175 50  0000 C CNN
-F 1 "Jack-DC" H 2757 1084 50  0000 C CNN
-F 2 "Connector_BarrelJack:BarrelJack_Horizontal" H 2750 810 50  0001 C CNN
-F 3 "~" H 2750 810 50  0001 C CNN
-	1    2700 850
-	0    -1   1    0
-$EndComp
-Wire Wire Line
-	2600 1700 2800 1700
-$Comp
-L Device:CP C1
-U 1 1 60904AC5
-P 2950 1700
-F 0 "C1" H 3068 1746 50  0000 L CNN
-F 1 "CP" H 3068 1655 50  0000 L CNN
-F 2 "Capacitor_THT:CP_Radial_D5.0mm_P2.00mm" H 2988 1550 50  0001 C CNN
-F 3 "~" H 2950 1700 50  0001 C CNN
-	1    2950 1700
-	0    -1   1    0
-$EndComp
-Wire Wire Line
-	2600 2800 1350 2800
-Wire Wire Line
-	2600 2800 2600 1700
-$Comp
 L Connector_Generic:Conn_01x04 J6
 U 1 1 609A3DBC
@@
 Connection ~ 6600 3600
 Wire Wire Line
-	1350 3600 3200 3600
-Connection ~ 3200 3600
-Connection ~ 2600 1700
-Connection ~ 3200 1150
-Wire Wire Line
-	3200 1150 3200 1700
-Wire Wire Line
-	2600 1150 2600 1700
-Wire Wire Line
-	3100 1700 3200 1700
-Connection ~ 3200 1700
-Wire Wire Line
-	3200 1700 3200 3600
-Wire Wire Line
-	3200 900  3200 1150
-Wire Wire Line
-	3200 900  3950 900
-Wire Wire Line
 	3850 4700 3850 5050
 Wire Wire Line
@@
 Wire Wire Line
 	4400 5050 4400 3600
-Connection ~ 4400 3600
 Wire Wire Line
 	4400 3600 5250 3600
 Wire Wire Line
-	3200 3600 4400 3600
-Wire Wire Line
 	2950 4000 2950 4400
 Wire Wire Line
@@
 Wire Wire Line
 	3850 3800 3850 4100
-Wire Wire Line
-	1350 3400 2750 3400
-Wire Wire Line
-	1350 3300 5350 3300
 Wire Wire Line
 	5350 5100 5350 3300
@@
 Wire Wire Line
 	10000 3100 10000 6350
+Connection ~ 4400 3600
+Wire Wire Line
+	1350 3300 3500 3300
+Wire Wire Line
+	1350 3400 2250 3400
+$Comp
+L Device:C C2
+U 1 1 60A632EF
+P 3500 3450
+F 0 "C2" H 3615 3496 50  0000 L CNN
+F 1 "100n" H 3615 3405 50  0000 L CNN
+F 2 "Capacitor_THT:C_Disc_D7.5mm_W4.4mm_P5.00mm" H 3538 3300 50  0001 C CNN
+F 3 "~" H 3500 3450 50  0001 C CNN
+	1    3500 3450
+	1    0    0    -1
+$EndComp
+Connection ~ 3500 3300
+Wire Wire Line
+	3500 3300 5350 3300
+Wire Wire Line
+	3500 3600 4400 3600
+$Comp
+L Device:C C1
+U 1 1 60A63A31
+P 2250 3550
+F 0 "C1" H 2365 3596 50  0000 L CNN
+F 1 "100n" H 2365 3505 50  0000 L CNN
+F 2 "Capacitor_THT:C_Disc_D7.5mm_W4.4mm_P5.00mm" H 2288 3400 50  0001 C CNN
+F 3 "~" H 2250 3550 50  0001 C CNN
+	1    2250 3550
+	1    0    0    -1
+$EndComp
+Connection ~ 2250 3400
+Wire Wire Line
+	2250 3400 2750 3400
+Wire Wire Line
+	1350 3600 2100 3600
+Wire Wire Line
+	2100 3600 2100 3700
+Wire Wire Line
+	2100 3700 2250 3700
+Wire Wire Line
+	2550 3700 2550 3600
+Wire Wire Line
+	2550 3600 3500 3600
+Connection ~ 2250 3700
+Wire Wire Line
+	2250 3700 2550 3700
+Connection ~ 3500 3600
 $EndSCHEMATC
